Commit message: dimmensions of cup correct, however, cup is shaky when in world need to figure out how to fix contacts, if incease radius of cup it solves this problem

File: tower/urdf/cups.urdf.xacro (robot description, xacro)
@@ -6,10 +6,9 @@
 <xacro:property name="length" value="${t['length']}"/>
 <xacro:property name="PI" value="3.1415926535897931" />
-    <!-- LEFT WHEEL -->
-  <link name="wheel_left_link">
+  <link name="cup1">
     <visual>
       <origin xyz="0 0 0" rpy="0 0 0"/>
       <geometry>
-        <cylinder radius= "1" length ="1" />
+        <cylinder radius= "${radius}" length ="${length}" />
       </geometry>
       <material name="black">
@@ -27,10 +26,10 @@
       <mass value="0.2" />
       <!-- mass = 0.2 in inertia eq -->
-      <inertia ixx="${0.2*(1/12)*(3*1**2 + 1**2)}" ixy="0" ixz="0"
-               iyy="${0.2*(1/12)*(3*1**2 + 1**2)}" iyz="0"
-               izz="${0.2*(1/2)*1**2}" />
+      <inertia ixx="${0.2*(1/12)*(3*radius**2 + length**2)}" ixy="0" ixz="0"
+               iyy="${0.2*(1/12)*(3*radius**2 + length**2)}" iyz="0"
+               izz="${0.2*(1/2)*radius**2}" />
       </inertial>
   </link>
-  <gazebo reference="wheel_left_link">
+  <gazebo reference="cup1">
     <mu1>1</mu1>
     <mu2>1</mu2>
@@ -38,32 +37,2 @@
   </gazebo>
 </robot>
-<!-- <link name="cup">
-  <visual>
-    <origin xyz="$0 0 0" rpy="$0 0 0" />
-    <geometry>
-      <cylinder radius="${radius}" length="${length}" />
-    </geometry>
-    <material name="blue_mat">
-         <color rgba="0 0 1 1" />
-    </material>
-  </visual>
-  <collision>
-    <origin xyz="0 0 0" rpy="0 0 0"/>
-    <geometry>
-      <cylinder radius="${radius}" length = "${length}"/>
-    </geometry>
-  </collision>
-  <inertial>
-    <origin xyz="0 0 0" />
-    <mass value="0.2" />
-    <inertia ixx="${0.2*(1/12)*(3*radius**2 + length**2)}" ixy="0" ixz="0"
-              iyy="${0.2*(1/12)*(3*radius**2 + length**2)}" iyz="0"
-              izz="${0.2*(1/2)*radius**2}" />
-  </inertial>
-</link>
-<gazebo reference="cup">
-  <mu1>1</mu1>
-  <mu2>1</mu2>
-  <material>Gazebo/Blue</material>
-</gazebo>
-</robot> -->
